Commit message: Add camera plugin, world and models

File: urdf/test_cameras.xacro (robot description, xacro)
@@ -10,4 +10,7 @@
     <color rgba="0 0 1 1" />
   </material>
+  <gazebo reference="base_link">
+    <material>Gazebo/Yellow</material>
+  </gazebo>
   <xacro:macro name="pan_camera" params="name y_offset">
     <link name="${name}_link">
@@ -63,4 +66,51 @@
       <child link="${name}_camera"/>
     </joint>
+    <gazebo reference="${name}_link">
+      <material>Gazebo/Blue</material>
+    </gazebo>
+    <gazebo reference="${name}_camera">
+      <material>Gazebo/Red</material>
+    </gazebo>
+    <!-- Gazebo camera plugin -->
+    <gazebo reference="${name}_camera">
+      <sensor type="camera" name="${name}_camera">
+        <update_rate>30.0</update_rate>
+        <camera name="${name}_camera">
+          <horizontal_fov>1.3962634</horizontal_fov>
+          <image>
+            <width>320</width>
+            <height>240</height>
+            <format>R8G8B8</format>
+          </image>
+          <clip>
+            <near>0.02</near>
+            <far>300</far>
+          </clip>
+          <noise>
+            <type>gaussian</type>
+              <!-- Noise is sampled independently per pixel on each frame.
+                That pixel's noise value is added to each of its color
+              channels, which at that point lie in the range [0,1]. -->
+            <mean>0.0</mean>
+            <stddev>0.007</stddev>
+          </noise>
+        </camera>
+        <plugin name="camera_controller" filename="libgazebo_ros_camera.so">
+          <alwaysOn>true</alwaysOn>
+          <updateRate>0.0</updateRate>
+          <cameraName>imove_camera/${name}_camera</cameraName>
+          <imageTopicName>image_raw</imageTopicName>
+          <cameraInfoTopicName>camera_info</cameraInfoTopicName>
+          <frameName>camera</frameName>
+          <hackBaseline>0.07</hackBaseline>
+          <distortionK1>0.0</distortionK1>
+          <distortionK2>0.0</distortionK2>
+          <distortionK3>0.0</distortionK3>
+          <distortionT1>0.0</distortionT1>
+          <distortionT2>0.0</distortionT2>
+        </plugin>
+        <visualize>true</visualize>
+      </sensor>
+    </gazebo>
   </xacro:macro>
   <link name="base_link">

Commit message: Add camera control

File: urdf/test_cameras.xacro (robot description, xacro)
@@ -72,4 +72,15 @@
       <material>Gazebo/Red</material>
     </gazebo>
+    <!-- Transmission block -->
+    <transmission name="tran_${name}">
+      <type>transmission_interface/SimpleTransmission</type>
+      <joint name="${name}_joint">
+        <hardwareInterface>hardware_interface/PositionJointInterface</hardwareInterface>
+      </joint>
+      <actuator name="motor_${name}">
+        <hardwareInterface>hardware_interface/PositionJointInterface</hardwareInterface>
+        <mechanicalReduction>1</mechanicalReduction>
+      </actuator>
+    </transmission>
     <!-- Gazebo camera plugin -->
     <gazebo reference="${name}_camera">
@@ -99,5 +110,5 @@
           <alwaysOn>true</alwaysOn>
           <updateRate>0.0</updateRate>
-          <cameraName>imove_camera/${name}_camera</cameraName>
+          <cameraName>test_camera/${name}_camera</cameraName>
           <imageTopicName>image_raw</imageTopicName>
           <cameraInfoTopicName>camera_info</cameraInfoTopicName>
@@ -135,3 +146,8 @@
   <xacro:pan_camera name="left" y_offset="0.25" />
   <xacro:pan_camera name="right" y_offset="-0.25" />
+  <gazebo>
+    <plugin name="gazebo_ros_control" filename="libgazebo_ros_control.so">
+      <robotNamespace>/test_cameras</robotNamespace>
+    </plugin>
+  </gazebo>
 </robot>
